Commit message: Add include guard to materials
Prevents material already defined errors when adding multiple types of camera to a robot

File: realsense2_description/urdf/_materials.urdf.xacro (robot description, xacro)
@@ -19,10 +19,14 @@
 This avoids the redefinition of materials in case multple cameras are imported.
 -->
-<robot>
-  <material name="aluminum">
-    <color rgba="0.5 0.5 0.5 1"/>
-  </material>
-  <material name="plastic">
-    <color rgba="0.1 0.1 0.1 1"/>
-  </material>
+<robot xmlns:xacro="http://ros.org/wiki/xacro">
+  <xacro:property name="realsense_materials_defined" default="false" />
+  <xacro:unless value="${realsense_materials_defined}">
+    <xacro:property name="realsense_materials_defined" value="true" />
+    <material name="aluminum">
+      <color rgba="0.5 0.5 0.5 1"/>
+    </material>
+    <material name="plastic">
+      <color rgba="0.1 0.1 0.1 1"/>
+    </material>
+ </xacro:unless>
 </robot>
